Commit message: feat: add spider & mammal flat config

File: legged_gym/resources/robots/el_4090/urdf/el_4090.urdf (robot description, URDF)
Before this commit: robot el_4090, 25 links, 24 joints
Joints:
- joint LB_HAA: limit lower=-1 upper=1 effort=80 velocity=15.8 -> lower=-5 upper=5 effort=80 velocity=15.8
- joint LB_HFE: limit lower=-1 upper=1 effort=80 velocity=15.8 -> lower=-5 upper=5 effort=80 velocity=15.8
- joint LB_KFE: limit lower=-1 upper=1 effort=80 velocity=15.8 -> lower=-5 upper=5 effort=80 velocity=15.8
- joint LF_HAA: limit lower=-1 upper=1 effort=80 velocity=15.8 -> lower=-5 upper=5 effort=80 velocity=15.8
- joint LF_HFE: limit lower=-1 upper=1 effort=80 velocity=15.8 -> lower=-5 upper=5 effort=80 velocity=15.8
- joint LF_KFE: limit lower=-1 upper=1 effort=80 velocity=15.8 -> lower=-5 upper=5 effort=80 velocity=15.8
- joint LM_HAA: limit lower=-1 upper=1 effort=80 velocity=15.8 -> lower=-5 upper=5 effort=80 velocity=15.8
- joint LM_HFE: limit lower=-1 upper=1 effort=80 velocity=15.8 -> lower=-5 upper=5 effort=80 velocity=15.8
- joint LM_KFE: limit lower=-1 upper=1 effort=80 velocity=15.8 -> lower=-5 upper=5 effort=80 velocity=15.8
- joint RB_HAA: limit lower=-1 upper=1 effort=80 velocity=15.8 -> lower=-5 upper=5 effort=80 velocity=15.8
- joint RB_HFE: limit lower=-1 upper=1 effort=80 velocity=15.8 -> lower=-5 upper=5 effort=80 velocity=15.8
- joint RB_KFE: limit lower=-1 upper=1 effort=80 velocity=15.8 -> lower=-5 upper=5 effort=80 velocity=15.8
- joint RF_HAA: limit lower=-1 upper=1 effort=80 velocity=15.8 -> lower=-5 upper=5 effort=80 velocity=15.8
- joint RF_HFE: limit lower=-1 upper=1 effort=80 velocity=15.8 -> lower=-5 upper=5 effort=80 velocity=15.8
- joint RF_KFE: limit lower=-1 upper=1 effort=80 velocity=15.8 -> lower=-5 upper=5 effort=80 velocity=15.8
- joint RM_HAA: limit lower=-1 upper=1 effort=80 velocity=15.8 -> lower=-5 upper=5 effort=80 velocity=15.8
- joint RM_HFE: limit lower=-1 upper=1 effort=80 velocity=15.8 -> lower=-5 upper=5 effort=80 velocity=15.8
- joint RM_KFE: limit lower=-1 upper=1 effort=80 velocity=15.8 -> lower=-5 upper=5 effort=80 velocity=15.8

Commit message: 2026/1/12  17:15

File: legged_gym/resources/robots/el_4090/urdf/el_4090.urdf (robot description, URDF)
Before this commit: robot el_4090, 25 links, 24 joints
Joints:
- joint LB_HAA: limit lower=-5 upper=5 effort=80 velocity=15.8 -> lower=-3 upper=3 effort=80 velocity=15.8
- joint LB_HFE: limit lower=-5 upper=5 effort=80 velocity=15.8 -> lower=-3 upper=3 effort=80 velocity=15.8
- joint LB_KFE: limit lower=-5 upper=5 effort=80 velocity=15.8 -> lower=-3 upper=3 effort=80 velocity=15.8
- joint LF_HAA: limit lower=-5 upper=5 effort=80 velocity=15.8 -> lower=-3 upper=3 effort=80 velocity=15.8
- joint LF_HFE: limit lower=-5 upper=5 effort=80 velocity=15.8 -> lower=-3 upper=3 effort=80 velocity=15.8
- joint LF_KFE: limit lower=-5 upper=5 effort=80 velocity=15.8 -> lower=-3 upper=3 effort=80 velocity=15.8
- joint LM_HAA: limit lower=-5 upper=5 effort=80 velocity=15.8 -> lower=-3 upper=3 effort=80 velocity=15.8
- joint LM_HFE: limit lower=-5 upper=5 effort=80 velocity=15.8 -> lower=-3 upper=3 effort=80 velocity=15.8
- joint LM_KFE: limit lower=-5 upper=5 effort=80 velocity=15.8 -> lower=-3 upper=3 effort=80 velocity=15.8
- joint RB_HAA: limit lower=-5 upper=5 effort=80 velocity=15.8 -> lower=-3 upper=3 effort=80 velocity=15.8
- joint RB_HFE: limit lower=-5 upper=5 effort=80 velocity=15.8 -> lower=-3 upper=3 effort=80 velocity=15.8
- joint RB_KFE: limit lower=-5 upper=5 effort=80 velocity=15.8 -> lower=-3 upper=3 effort=80 velocity=15.8
- joint RF_HAA: limit lower=-5 upper=5 effort=80 velocity=15.8 -> lower=-3 upper=3 effort=80 velocity=15.8
- joint RF_HFE: limit lower=-5 upper=5 effort=80 velocity=15.8 -> lower=-3 upper=3 effort=80 velocity=15.8
- joint RF_KFE: limit lower=-5 upper=5 effort=80 velocity=15.8 -> lower=-3 upper=3 effort=80 velocity=15.8
- joint RM_HAA: limit lower=-5 upper=5 effort=80 velocity=15.8 -> lower=-3 upper=3 effort=80 velocity=15.8
- joint RM_HFE: limit lower=-5 upper=5 effort=80 velocity=15.8 -> lower=-3 upper=3 effort=80 velocity=15.8
- joint RM_KFE: limit lower=-5 upper=5 effort=80 velocity=15.8 -> lower=-3 upper=3 effort=80 velocity=15.8

Commit message: 完善ATACOM接口，修改safe版本obs数量，将u_mu加入obs，调整关节限位和机身限位。

File: legged_gym/resources/robots/el_4090/urdf/el_4090.urdf (robot description, URDF)
Before this commit: robot el_4090, 25 links, 24 joints
Links:
- link BASE: mass 7.44160057363592 -> 10
- link LB_HIP: mass 1.1161 -> 1.8161
- link LB_THIGH: mass 1.0012 -> 2.4012
- link LF_HIP: mass 1.1161 -> 1.8161
- link LF_THIGH: mass 1.0012 -> 2.4012
- link LM_HIP: mass 1.1161 -> 1.8161
- link LM_THIGH: mass 1.0012 -> 2.4012
- link RB_HIP: mass 1.1161 -> 1.8161
- link RB_THIGH: mass 1.3913 -> 2.7913
- link RF_HIP: mass 1.11609830949325 -> 1.81609830949325
- link RF_THIGH: mass 1.00124210184093 -> 2.40124210184093
- link RM_HIP: mass 1.1161 -> 1.8161
- link RM_THIGH: mass 1.0012 -> 2.4012

Commit message: 修改了el_4090的安全环境和正常环境的代码和urdf文件。

File: legged_gym/resources/robots/el_4090/urdf/el_4090.urdf (robot description, URDF)
Before this commit: robot el_4090, 25 links, 24 joints
Joints:
- joint LB_HAA: limit lower=-3 upper=3 effort=80 velocity=15.8 -> lower=-1.57 upper=1.57 effort=80 velocity=15.8
- joint LB_HFE: limit lower=-3 upper=3 effort=80 velocity=15.8 -> lower=-1.57 upper=1.57 effort=80 velocity=15.8
- joint LB_KFE: limit lower=-3 upper=3 effort=80 velocity=15.8 -> lower=-1.57 upper=1.57 effort=80 velocity=15.8
- joint LF_HAA: limit lower=-3 upper=3 effort=80 velocity=15.8 -> lower=-1.57 upper=1.57 effort=80 velocity=15.8
- joint LF_HFE: limit lower=-3 upper=3 effort=80 velocity=15.8 -> lower=-1.57 upper=1.57 effort=80 velocity=15.8
- joint LF_KFE: limit lower=-3 upper=3 effort=80 velocity=15.8 -> lower=-1.57 upper=1.57 effort=80 velocity=15.8
- joint LM_HAA: limit lower=-3 upper=3 effort=80 velocity=15.8 -> lower=-1.57 upper=1.57 effort=80 velocity=15.8
- joint LM_HFE: limit lower=-3 upper=3 effort=80 velocity=15.8 -> lower=-1.57 upper=1.57 effort=80 velocity=15.8
- joint LM_KFE: limit lower=-3 upper=3 effort=80 velocity=15.8 -> lower=-1.57 upper=1.57 effort=80 velocity=15.8
- joint RB_HAA: limit lower=-3 upper=3 effort=80 velocity=15.8 -> lower=-1.57 upper=1.57 effort=80 velocity=15.8
- joint RB_HFE: limit lower=-3 upper=3 effort=80 velocity=15.8 -> lower=-1.57 upper=1.57 effort=80 velocity=15.8
- joint RB_KFE: limit lower=-3 upper=3 effort=80 velocity=15.8 -> lower=-1.57 upper=1.57 effort=80 velocity=15.8
- joint RF_HAA: limit lower=-3 upper=3 effort=80 velocity=15.8 -> lower=-1.57 upper=1.57 effort=80 velocity=15.8
- joint RF_HFE: limit lower=-3 upper=3 effort=80 velocity=15.8 -> lower=-1.57 upper=1.57 effort=80 velocity=15.8
- joint RF_KFE: limit lower=-3 upper=3 effort=80 velocity=15.8 -> lower=-1.57 upper=1.57 effort=80 velocity=15.8
- joint RM_HAA: limit lower=-3 upper=3 effort=80 velocity=15.8 -> lower=-1.57 upper=1.57 effort=80 velocity=15.8
- joint RM_HFE: limit lower=-3 upper=3 effort=80 velocity=15.8 -> lower=-1.57 upper=1.57 effort=80 velocity=15.8
- joint RM_KFE: limit lower=-3 upper=3 effort=80 velocity=15.8 -> lower=-1.57 upper=1.57 effort=80 velocity=15.8
